File: sk6805_grid.kicad_pcb (KiCad board)
At the start: 2 copper layers, 26.7 x 21.6 mm, 73 parts

Commit message: Add logo and version stamp
Parts:
- added REF**: Logo_WM, Symbol:Logo_WM, B.Cu at (100.8, 78.5)
Other:
- board text added: "v0.0.0 04/22/20"
Changed lines of the file:
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@@
   (general
     (thickness 1.6)
-    (drawings 4)
+    (drawings 5)
     (tracks 790)
     (zones 0)
-    (modules 73)
+    (modules 74)
     (nets 68)
   )
@@
   )
   (setup
-    (last_trace_width 0.2)
+    (last_trace_width 0.25)
     (user_trace_width 0.2)
     (trace_clearance 0.2)
@@
     (aux_axis_origin 0 0)
     (grid_origin 93.92 68.38)
-    (visible_elements FFFFFF7F)
+    (visible_elements 7FFFFFFF)
     (pcbplotparams
       (layerselection 0x010fc_ffffffff)
@@
     (add_net "Net-(D7-Pad1)")
   )
+  (module Symbol:Logo_WM (layer B.Cu)
+    (at 100.7907 78.54)
+    (fp_text reference REF** (at 0 2.286) (layer B.SilkS) hide
+      (effects (font (size 1 1) (thickness 0.15)) (justify mirror))
+    )
+    (fp_text value Logo_WM (at 0 -2.032) (layer B.Fab)
+      (effects (font (size 1 1) (thickness 0.15)) (justify mirror))
+    )
+    (fp_poly (pts (xy 0.635 0) (xy 1.905 0) (xy 1.27 -1.143)) (layer B.SilkS) (width 0.1))
+    (fp_poly (pts (xy -0.635 0) (xy 0.635 0) (xy 0 1.143)) (layer B.SilkS) (width 0.1))
+    (fp_poly (pts (xy -1.905 0) (xy -0.635 0) (xy -1.27 -1.143)) (layer B.SilkS) (width 0.1))
+    (fp_line (start 1.905 0) (end 2.54 -1.143) (layer B.SilkS) (width 0.12))
+    (fp_line (start 2.54 1.143) (end 1.905 0) (layer B.SilkS) (width 0.12))
+    (fp_line (start -2.54 -1.143) (end -1.905 0) (layer B.SilkS) (width 0.12))
+    (fp_line (start -1.905 0) (end -2.54 1.143) (layer B.SilkS) (width 0.12))
+    (fp_line (start -0.635 0) (end -1.27 1.143) (layer B.SilkS) (width 0.12))
+    (fp_line (start -1.905 0) (end -1.27 -1.143) (layer B.SilkS) (width 0.12))
+    (fp_line (start -1.27 1.143) (end -1.905 0) (layer B.SilkS) (width 0.12))
+    (fp_line (start -1.27 -1.143) (end -0.635 0) (layer B.SilkS) (width 0.12))
+    (fp_line (start 1.27 1.143) (end 0.635 0) (layer B.SilkS) (width 0.12))
+    (fp_line (start 0.635 0) (end 1.27 -1.143) (layer B.SilkS) (width 0.12))
+    (fp_line (start 1.27 -1.143) (end 1.905 0) (layer B.SilkS) (width 0.12))
+    (fp_line (start 1.905 0) (end 1.27 1.143) (layer B.SilkS) (width 0.12))
+    (fp_line (start 0.635 0) (end 0 1.143) (layer B.SilkS) (width 0.12))
+    (fp_line (start 0 -1.143) (end 0.635 0) (layer B.SilkS) (width 0.12))
+    (fp_line (start -0.635 0) (end 0 -1.143) (layer B.SilkS) (width 0.12))
+    (fp_line (start 0 1.143) (end -0.635 0) (layer B.SilkS) (width 0.12))
+  )
   (module LED_SMD:LED_SK6805_PLCC4_1.5x1.5mm_P0.65mm (layer F.Cu)
     (at 99 68.38 180)
@@
     )
   )
+  (gr_text "v0.0.0\n04/22/20" (at 110.5316 77.1176 180) (layer B.SilkS)
+    (effects (font (size 1.5 1.5) (thickness 0.3)) (justify right mirror))
+  )
   (gr_line (start 86.935 88.065) (end 86.935 66.475) (layer Edge.Cuts) (width 0.05))
